File: #100 Robot/#160 PCB/Eagle/PCB_Robotique_V3.brd (EAGLE design)
At the start: 127 x 58.9 mm, 21 parts, among them X1 057-034-1, X11 057-006-1, X12 057-006-1, X13 057-014-1, X15 057-006-1, X2 057-006-1, X3 057-010-1, X4 332-02, X5 057-034-1, X7 057-010-1

Commit message: Modification PCB_V3
Parts:
- removed X12, X2: 057-006-1, con-panduit:057-006-1
- removed X4: 332-02, con-garry:332-02
- added 5V: 057-006-1, con-panduit:057-006-1
- added PWM_LANCEUR_MAN: MA01-1, connecteurs_males:MA01-1
- added TRIEUR_DIODE: (no value), connecteurs_males:MA03-1
- R1: value (none) -> 100K
- R2: value (none) -> 220
- moved X6 36.8 mm to (119.3, 6.35)
- renumbered X1 to MYRIO_PORT_B, X11 to TRIEUR_PWM, X13 to ROUE, X15 to LANCEUR, X3 to LIDAR, X5 to MYRIO_PORT_A
Connections:
- removed net N$1 (its old number): J2.4, MYRIO_PORT_A.28
- removed net N$10: J2.8, MYRIO_PORT_A.20
- removed net N$15: J3.8, MYRIO_PORT_A.33
- removed net N$21: J7.5, MYRIO_PORT_B.8
- removed net N$23: J7.3, MYRIO_PORT_B.12
- removed net N$31: J4.1, MYRIO_PORT_A.1
- removed net N$33: J7.1, MYRIO_PORT_B.16
- removed net N$34: J8.6, MYRIO_PORT_B.24
- removed net N$36: J8.4, MYRIO_PORT_B.28
- removed net N$37: J8.3, MYRIO_PORT_B.30
- removed net N$4: J2.6, MYRIO_PORT_A.24
- removed net N$40: J9.9, MYRIO_PORT_B.33
- removed net N$51: X12.4
- removed net N$52: X12.6
- removed net N$6: J5.2, MYRIO_PORT_A.16
- removed net SUIVEUR_A: J6.2, MYRIO_PORT_B.3, R1.2, X12.1
- new net ALIM_3.3V: J3.8, J9.9, MYRIO_PORT_A.33, MYRIO_PORT_B.33
- new net DIODE_EMETEUR: J6.2, MYRIO_PORT_B.3, R1.2, TRIEUR_DIODE.1
- net +5V: now also 5V.2, 5V.4, 5V.6; no longer X2.2, X2.4, X2.6
- net ALIM_+5V: now also J4.1, MYRIO_PORT_A.1, TRIEUR_DIODE.2; no longer X12.3
- net A_MODIF_POUR_DATA_MOTEUR_1.5V: now also TRIEUR_DIODE.3; no longer X12.5
- net GND: now also 5V.1, 5V.3, 5V.5, J2.4, J2.6, J2.8, J5.2, J7.1, J7.3, J7.5, J8.3, J8.4, J8.6, MYRIO_PORT_A.16, MYRIO_PORT_A.20, MYRIO_PORT_A.24, MYRIO_PORT_A.28, MYRIO_PORT_B.12, MYRIO_PORT_B.16, MYRIO_PORT_B.24, MYRIO_PORT_B.28, MYRIO_PORT_B.30, MYRIO_PORT_B.8; no longer X2.1, X2.3, X2.5
- net PWM_LANCEUR_MAN: now also PWM_LANCEUR_MAN.1; no longer X4.2
Routing:
- net GND: track 0.00 -> 91.4 mm
- net SUIVEUR_A: track 57.8 -> 0.00 mm
- net DIODE_EMETEUR: track 0.00 -> 57.5 mm
- net +5V: track 185.5 -> 205.5 mm
- net ALIM_3.3V: track 0.00 -> 15.2 mm
- net ALIM_+5V: track 40.0 -> 47.6 mm
- net N$6: track 7.62 -> 0.00 mm
- net N$40: track 7.62 -> 0.00 mm
- net N$4: track 7.62 -> 0.00 mm
- net N$37: track 7.62 -> 0.00 mm
- net N$36: track 7.62 -> 0.00 mm
- net N$34: track 7.62 -> 0.00 mm
- net N$33: track 7.62 -> 0.00 mm
- net N$31: track 7.62 -> 0.00 mm
- net N$23: track 7.62 -> 0.00 mm
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
Commit message: Update PCB V3 + Gestion de Projet
Parts:
- removed X7: 057-010-1, con-panduit:057-010-1
- added X1: 22-23-2031, con-molex:22-23-2031
- added X2: 22-23-2041, con-molex:22-23-2041
- R1: value 100K -> 15K
- R2: value 220 -> 180
- moved PWM_LANCEUR_MAN 1.79 mm to (5.60, 35.2), turned to 90 degrees
Connections:
- net A_MODIF_POUR_DATA_MOTEUR_1.5V renamed DIODE
- removed net N$1: J5.6, MYRIO_PORT_A.8
- removed net N$2: J5.4, MYRIO_PORT_A.12
- net +5V: now also ROUE.12, X1.2, X2.3; no longer ROUE.4, X7.5, X7.6
- net BRAS_PWM: now also X1.1; no longer X7.3
- net GND: now also J5.4, J5.6, MYRIO_PORT_A.12, MYRIO_PORT_A.8, ROUE.10, ROUE.4, X1.3, X2.4; no longer ROUE.12, ROUE.6, X7.7, X7.8
- net ROUE_MOTEUR_1_ENCODEUR_A: now also ROUE.13; no longer ROUE.1
- net ROUE_MOTEUR_1_ENCODEUR_B: now also ROUE.11; no longer ROUE.3
- net ROUE_MOTEUR_1_PWM_0: now also ROUE.5; no longer ROUE.9
- net ROUE_MOTEUR_2_ENCODEUR_A: now also ROUE.9; no longer ROUE.5
- net ROUE_MOTEUR_2_PWM_1: now also ROUE.3; no longer ROUE.11
- net SUIVEUR_I2C_SCL: now also X2.2; no longer X7.4
- net SUIVEUR_IDC_SDA: now also X2.1; no longer X7.2
Routing:
- net BRAS_PWM: track 109.9 -> 41.4 mm, vias 1 -> 0
- net ROUE_MOTEUR_2_PWM_1: track 45.6 -> 70.7 mm, vias 1 -> 2
- net GND: track 91.4 -> 106.7 mm
- net SUIVEUR_IDC_SDA: track 21.9 -> 35.0 mm
- net SUIVEUR_I2C_SCL: track 21.9 -> 35.0 mm
- net ROUE_MOTEUR_1_ENCODEUR_A: track 59.6 -> 46.9 mm, vias 2 -> 1
- net ROUE_MOTEUR_1_ENCODEUR_B: track 55.1 -> 44.0 mm, vias 2 -> 1
- net ROUE_MOTEUR_2_ENCODEUR_A: track 114.1 -> 104.3 mm
- net N$2: track 7.62 -> 0.00 mm
- net N$1: track 7.62 -> 0.00 mm
- net ROUE_MOTEUR_2_ENCODEUR_B: track 102.2 -> 106.9 mm, vias 0 -> 2
- net ROUE_MOTEUR_1_PWM_0: track 56.5 -> 60.4 mm
- net PWM_LANCEUR_MAN: track 9.89 -> 8.20 mm
- net +5V: track 205.5 -> 206.6 mm, vias 1 -> 0
- net AGND: track 30.5 -> 31.0 mm
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
Commit message: Auto stash before merge of "Dev" and "origin/Dev"
Parts:
- renumbered X1 to BRAS, X2 to SUIVEUR, X6 to 5V_EXTERNE
Routing:
- net 4B: track 7.62 -> 0.00 mm
Changed lines of the file:
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@@
 <layer number="17" name="Pads" color="2" fill="1" visible="yes" active="yes"/>
 <layer number="18" name="Vias" color="2" fill="1" visible="yes" active="yes"/>
-<layer number="19" name="Unrouted" color="6" fill="1" visible="yes" active="yes"/>
+<layer number="19" name="Unrouted" color="6" fill="1" visible="no" active="yes"/>
 <layer number="20" name="Dimension" color="15" fill="1" visible="yes" active="yes"/>
 <layer number="21" name="tPlace" color="7" fill="1" visible="yes" active="yes"/>
 <layer number="22" name="bPlace" color="7" fill="1" visible="yes" active="yes"/>
-<layer number="23" name="tOrigins" color="15" fill="1" visible="yes" active="yes"/>
-<layer number="24" name="bOrigins" color="15" fill="1" visible="yes" active="yes"/>
+<layer number="23" name="tOrigins" color="15" fill="1" visible="no" active="yes"/>
+<layer number="24" name="bOrigins" color="15" fill="1" visible="no" active="yes"/>
 <layer number="25" name="tNames" color="7" fill="1" visible="yes" active="yes"/>
 <layer number="26" name="bNames" color="7" fill="1" visible="yes" active="yes"/>
 <layer number="27" name="tValues" color="7" fill="1" visible="yes" active="yes"/>
-<layer number="28" name="bValues" color="7" fill="1" visible="yes" active="yes"/>
+<layer number="28" name="bValues" color="7" fill="1" visible="no" active="yes"/>
 <layer number="29" name="tStop" color="7" fill="3" visible="no" active="yes"/>
 <layer number="30" name="bStop" color="7" fill="6" visible="no" active="yes"/>
@@
 <attribute name="VALUE" x="106.7306" y="19.215" size="1.27" layer="27" ratio="10"/>
 </element>
-<element name="X6" library="isenproject" package="KK-156-2" value="" x="119.35" y="6.35" smashed="yes" rot="R270">
+<element name="5V_EXTERNE" library="isenproject" package="KK-156-2" value="" x="119.35" y="6.35" smashed="yes" rot="R270">
 <attribute name="MF" value="" x="31.72" y="-27.94" size="1.778" layer="27" rot="R270" display="off"/>
 <attribute name="MPN" value="" x="31.72" y="-27.94" size="1.778" layer="27" rot="R270" display="off"/>
@@
 </element>
 <element name="PWM_LANCEUR_MAN" library="connecteurs_males" package="MA01-1" value="MA01-1" x="5.6" y="35.2" rot="R90"/>
-<element name="X1" library="con-molex" library_urn="urn:adsk.eagle:library:165" package="22-23-2031" value="22-23-2031" x="52.8" y="25.6" rot="R180">
+<element name="BRAS" library="con-molex" library_urn="urn:adsk.eagle:library:165" package="22-23-2031" value="22-23-2031" x="52.8" y="25.6" rot="R180">
 <attribute name="MF" value="MOLEX" x="52.8" y="25.6" size="1.778" layer="27" rot="R180" display="off"/>
 <attribute name="MPN" value="22-23-2031" x="52.8" y="25.6" size="1.778" layer="27" rot="R180" display="off"/>
@@
 <attribute name="OC_NEWARK" value="30C0862" x="52.8" y="25.6" size="1.778" layer="27" rot="R180" display="off"/>
 </element>
-<element name="X2" library="con-molex" library_urn="urn:adsk.eagle:library:165" package="22-23-2041" value="22-23-2041" x="21.6" y="5.6">
+<element name="SUIVEUR" library="con-molex" library_urn="urn:adsk.eagle:library:165" package="22-23-2041" value="22-23-2041" x="21.6" y="5.6">
 <attribute name="MF" value="MOLEX" x="21.6" y="5.6" size="1.778" layer="27" display="off"/>
 <attribute name="MPN" value="22-23-2041" x="21.6" y="5.6" size="1.778" layer="27" display="off"/>
@@
 <signals>
 <signal name="GND">
-<contactref element="X6" pad="2"/>
+<contactref element="5V_EXTERNE" pad="2"/>
 <contactref element="MYRIO_PORT_A" pad="30"/>
 <contactref element="TRIEUR_PWM" pad="1"/>
@@
 <contactref element="J5" pad="4"/>
 <wire x1="45.72" y1="33.02" x2="45.72" y2="40.64" width="0.6096" layer="16"/>
-<contactref element="X1" pad="3"/>
-<contactref element="X2" pad="4"/>
+<contactref element="BRAS" pad="3"/>
+<contactref element="SUIVEUR" pad="4"/>
 </signal>
 <signal name="+5V">
@@
 <contactref element="TRIEUR_PWM" pad="3"/>
 <contactref element="TRIEUR_PWM" pad="4"/>
-<contactref element="X6" pad="1"/>
+<contactref element="5V_EXTERNE" pad="1"/>
 <contactref element="LANCEUR" pad="4"/>
 <contactref element="5V" pad="4"/>
@@
 <wire x1="80.3" y1="4.98" x2="80.12" y2="4.8" width="0.6096" layer="16"/>
 <contactref element="ROUE" pad="12"/>
-<contactref element="X1" pad="2"/>
-<contactref element="X2" pad="3"/>
+<contactref element="BRAS" pad="2"/>
+<contactref element="SUIVEUR" pad="3"/>
 <wire x1="100.33" y1="5.08" x2="100.33" y2="7.62" width="1.016" layer="16"/>
 <wire x1="100.33" y1="7.62" x2="100.33" y2="9.13" width="1.016" layer="16"/>
@@
 <contactref element="J2" pad="2"/>
 <wire x1="20.32" y1="40.64" x2="20.32" y2="33.02" width="0.6096" layer="16"/>
-<contactref element="X2" pad="2"/>
+<contactref element="SUIVEUR" pad="2"/>
 <wire x1="20.32" y1="5.61" x2="20.33" y2="5.6" width="0.6096" layer="16"/>
 <wire x1="20.32" y1="33.02" x2="20.32" y2="5.61" width="0.6096" layer="16"/>
@@
 <contactref element="J2" pad="1"/>
 <wire x1="17.78" y1="40.64" x2="17.78" y2="33.02" width="0.6096" layer="16"/>
-<contactref element="X2" pad="1"/>
+<contactref element="SUIVEUR" pad="1"/>
 <wire x1="17.78" y1="5.61" x2="17.79" y2="5.6" width="0.6096" layer="16"/>
 <wire x1="17.78" y1="33.02" x2="17.78" y2="5.61" width="0.6096" layer="16"/>
@@
 <contactref element="J9" pad="8"/>
 <wire x1="77.47" y1="50.8" x2="77.47" y2="43.18" width="0.6096" layer="16"/>
-<contactref element="X1" pad="1"/>
+<contactref element="BRAS" pad="1"/>
 <wire x1="77.47" y1="43.18" x2="75.05" y2="45.6" width="0.6096" layer="1"/>
 <wire x1="75.05" y1="45.6" x2="72.8" y2="45.6" width="0.6096" layer="1"/>
@@
 <contactref element="MYRIO_PORT_B" pad="4"/>
 <contactref element="J7" pad="7"/>
-<wire x1="113.03" y1="33.02" x2="113.03" y2="40.64" width="0.6096" layer="16"/>
+<wire x1="113.03" y1="33.02" x2="113.03" y2="40.64" width="0" layer="19" extent="1-1"/>
 </signal>
 <signal name="AGND">

Commit message: Update PCB et Datasheet PCB
Connections:
- net SUIVEUR_IDC_SDA renamed SUIVEUR_I2C_SDA
Changed lines of the file:
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@@
 <wire x1="20.32" y1="33.02" x2="20.32" y2="5.61" width="0.6096" layer="16"/>
 </signal>
-<signal name="SUIVEUR_IDC_SDA">
+<signal name="SUIVEUR_I2C_SDA">
 <contactref element="MYRIO_PORT_A" pad="34"/>
 <contactref element="J2" pad="1"/>
