File: #100 Robot/#160 PCB/Eagle/PCB_Robotique_V3.sch (EAGLE design)
At the start: 21 parts, among them X1 057-034-1, X11 057-006-1, X12 057-006-1, X13 057-014-1, X15 057-006-1, X2 057-006-1, X3 057-010-1, X4 332-02, X5 057-034-1, X7 057-010-1

Commit message: Modification PCB_V3
Parts:
- removed X1: 057-034-1, con-panduit:057-034-1
- removed X11, X12: 057-006-1, con-panduit:057-006-1
- removed X13: 057-014-1, con-panduit:057-014-1
- removed X4: 332-02, con-garry:332-02
- added MYRIO_PORT_B: 057-034-1, con-panduit:057-034-1
- added PWM_LANCEUR_MAN: MA01-1, connecteurs_males:MA01-1
- added ROUE: 057-014-1, con-panduit:057-014-1
- added TRIEUR_DIODE: (no value), connecteurs_males:MA03-1
- added TRIEUR_PWM: 057-006-1, con-panduit:057-006-1
- R1: value (none) -> 100K
- R2: value (none) -> 220
- renumbered X15 to LANCEUR, X2 to 5V, X3 to LIDAR, X5 to MYRIO_PORT_A
Connections:
- removed net N$1 (its old number): J2.4, MYRIO_PORT_A-28.S
- removed net N$10: J2.8, MYRIO_PORT_A-20.S
- removed net N$15: J3.8, MYRIO_PORT_A-33.S
- removed net N$21: J7.5, X1-8.S
- removed net N$23: J7.3, X1-12.S
- removed net N$31: J4.1, MYRIO_PORT_A-1.S
- removed net N$33: J7.1, X1-16.S
- removed net N$34: J8.6, X1-24.S
- removed net N$36: J8.4, X1-28.S
- removed net N$37: J8.3, X1-30.S
- removed net N$4: J2.6, MYRIO_PORT_A-24.S
- removed net N$40: J9.9, X1-33.S
- removed net N$51: X12-4.S
- removed net N$52: X12-6.S
- removed net N$6: J5.2, MYRIO_PORT_A-16.S
- removed net SUIVEUR_A: J6.2, R1.2, X1-3.S, X12-1.S
- new net ALIM_3.3V: J3.8, J9.9, MYRIO_PORT_A-33.S, MYRIO_PORT_B-33.S
- new net DIODE_EMETEUR: J6.2, MYRIO_PORT_B-3.S, R1.2, TRIEUR_DIODE.1
- net +5V: now also ROUE-4.S, TRIEUR_PWM-3.S, TRIEUR_PWM-4.S; no longer X11-3.S, X11-4.S, X13-4.S
- net 4B: now also MYRIO_PORT_B-4.S; no longer X1-4.S
- net AGND: now also MYRIO_PORT_B-6.S; no longer X1-6.S
- net ALIM_+5V: now also J4.1, MYRIO_PORT_A-1.S, MYRIO_PORT_B-1.S, TRIEUR_DIODE.2; no longer X1-1.S, X12-3.S
- net A_MODIF_POUR_DATA_MOTEUR_1.5V: now also TRIEUR_DIODE.3; no longer X12-5.S
- net BRAS_PWM: now also MYRIO_PORT_B-31.S; no longer X1-31.S
- net GND: now also J2.4, J2.6, J2.8, J5.2, J7.1, J7.3, J7.5, J8.3, J8.4, J8.6, MYRIO_PORT_A-16.S, MYRIO_PORT_A-20.S, MYRIO_PORT_A-24.S, MYRIO_PORT_A-28.S, MYRIO_PORT_B-12.S, MYRIO_PORT_B-16.S, MYRIO_PORT_B-20.S, MYRIO_PORT_B-24.S, MYRIO_PORT_B-28.S, MYRIO_PORT_B-30.S, MYRIO_PORT_B-8.S, ROUE-12.S, ROUE-6.S, TRIEUR_PWM-1.S, TRIEUR_PWM-2.S; no longer X1-20.S, X11-1.S, X11-2.S, X13-12.S, X13-6.S
- net LIDAR_RX: now also MYRIO_PORT_B-14.S; no longer X1-14.S
- net LIDAR_TX: now also MYRIO_PORT_B-10.S; no longer X1-10.S
- net MOTOCTL: now also MYRIO_PORT_B-26.S; no longer X1-26.S
- net N$38: now also MYRIO_PORT_B-32.S; no longer X1-32.S
- net N$39: now also MYRIO_PORT_B-34.S; no longer X1-34.S
- net N$41: now also MYRIO_PORT_B-25.S; no longer X1-25.S
- net N$42: now also MYRIO_PORT_B-23.S; no longer X1-23.S
- net N$43: now also MYRIO_PORT_B-21.S; no longer X1-21.S
- net N$44: now also MYRIO_PORT_B-19.S; no longer X1-19.S
- net N$45: now also MYRIO_PORT_B-17.S; no longer X1-17.S
- net N$46: now also MYRIO_PORT_B-15.S; no longer X1-15.S
- net N$47: now also MYRIO_PORT_B-9.S; no longer X1-9.S
- net N$48: now also MYRIO_PORT_B-7.S; no longer X1-7.S
- net N$49: now also MYRIO_PORT_B-5.S; no longer X1-5.S
- net N$7: now also MYRIO_PORT_B-2.S; no longer X1-2.S
- net PWM_LANCEUR_MAN: now also PWM_LANCEUR_MAN.1; no longer X4-2.S
- net ROUE_MOTEUR_1_ENCODEUR_A: now also ROUE-1.S; no longer X13-1.S
- net ROUE_MOTEUR_1_ENCODEUR_B: now also ROUE-3.S; no longer X13-3.S
- net ROUE_MOTEUR_1_PWM_0: now also ROUE-9.S; no longer X13-9.S
- net ROUE_MOTEUR_2_ENCODEUR_A: now also MYRIO_PORT_B-18.S, ROUE-5.S; no longer X1-18.S, X13-5.S
- net ROUE_MOTEUR_2_ENCODEUR_B: now also MYRIO_PORT_B-22.S, ROUE-7.S; no longer X1-22.S, X13-7.S
- net ROUE_MOTEUR_2_PWM_1: now also ROUE-11.S; no longer X13-11.S
- net TRIEUR_PWM_0: now also MYRIO_PORT_B-27.S, TRIEUR_PWM-6.S; no longer X1-27.S, X11-6.S
- net TRIEUR_PWM_2: now also MYRIO_PORT_B-29.S, TRIEUR_PWM-5.S; no longer X1-29.S, X11-5.S
- net ULTRA_D1: now also MYRIO_PORT_B-11.S; no longer X1-11.S
- net ULTRA_D2: now also MYRIO_PORT_B-13.S; no longer X1-13.S
Other:
- moved on the sheet: J6, J7, J8, J9, R1, R2, X7-1, X7-10, X7-2, X7-3, X7-4, X7-5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

Commit message: Update PCB V3 + Gestion de Projet
Parts:
- removed X7: 057-010-1, con-panduit:057-010-1
- added X1: 22-23-2031, con-molex:22-23-2031
- added X2: 22-23-2041, con-molex:22-23-2041
- R1: value 100K -> 15K
- R2: value 220 -> 180
Connections:
- net A_MODIF_POUR_DATA_MOTEUR_1.5V renamed DIODE
- removed net N$1: J5.6, MYRIO_PORT_A-8.S
- removed net N$2: J5.4, MYRIO_PORT_A-12.S
- net +5V: now also ROUE-12.S, X1-2.S, X2-3.S; no longer ROUE-4.S, X7-5.S, X7-6.S
- net BRAS_PWM: now also X1-1.S; no longer X7-3.S
- net GND: now also J5.4, J5.6, MYRIO_PORT_A-12.S, MYRIO_PORT_A-8.S, ROUE-10.S, ROUE-4.S, X1-3.S, X2-4.S; no longer ROUE-12.S, ROUE-6.S, X7-7.S, X7-8.S
- net ROUE_MOTEUR_1_ENCODEUR_A: now also ROUE-13.S; no longer ROUE-1.S
- net ROUE_MOTEUR_1_ENCODEUR_B: now also ROUE-11.S; no longer ROUE-3.S
- net ROUE_MOTEUR_1_PWM_0: now also ROUE-5.S; no longer ROUE-9.S
- net ROUE_MOTEUR_2_ENCODEUR_A: now also ROUE-9.S; no longer ROUE-5.S
- net ROUE_MOTEUR_2_PWM_1: now also ROUE-3.S; no longer ROUE-11.S
- net SUIVEUR_I2C_SCL: now also X2-2.S; no longer X7-4.S
- net SUIVEUR_IDC_SDA: now also X2-1.S; no longer X7-2.S
Other:
- note added: "ATTENTION : Les pins sont placées en top view. Dans la réalité les pins sont connectées au reste du robot par le dessous"
- note added: "Les VIA: Diameter=auto; Drill= 0,6096"
- note added: "Les routes de signaux sont tracées en 0,6096 mm = 0,024 Pouce"
- moved on the sheet: 5V-1, 5V-2, 5V-3, 5V-4, 5V-5, 5V-6, ROUE-1, ROUE-10, ROUE-11, ROUE-12, ROUE-13, ROUE-14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

Commit message: Auto stash before merge of "Dev" and "origin/Dev"
Parts:
- removed X1: 22-23-2031, con-molex:22-23-2031
- removed X2: 22-23-2041, con-molex:22-23-2041
- added BRAS: 22-23-2031, con-molex:22-23-2031
- added SUIVEUR: 22-23-2041, con-molex:22-23-2041
- renumbered X6 to 5V_EXTERNE
Connections:
- net +5V: now also BRAS-2.S, SUIVEUR-3.S; no longer X1-2.S, X2-3.S
- net BRAS_PWM: now also BRAS-1.S; no longer X1-1.S
- net GND: now also BRAS-3.S, SUIVEUR-4.S; no longer X1-3.S, X2-4.S
- net SUIVEUR_I2C_SCL: now also SUIVEUR-2.S; no longer X2-2.S
- net SUIVEUR_IDC_SDA: now also SUIVEUR-1.S; no longer X2-1.S
Other:
- note added: "Les routes de POWER sont tracées en 1,016 mm = 0,040 Pouce"
- moved on the sheet: MYRIO_PORT_A-1, MYRIO_PORT_A-10, MYRIO_PORT_A-11, MYRIO_PORT_A-12, MYRIO_PORT_A-13, MYRIO_PORT_A-14, MYRIO_PORT_A-15, MYRIO_PORT_A-16, MYRIO_PORT_A-17, MYRIO_PORT_A-18, MYRIO_PORT_A-19, MYRIO_PORT_A-2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

Commit message: Update PCB et Datasheet PCB
Connections:
- net SUIVEUR_IDC_SDA renamed SUIVEUR_I2C_SDA
Changed lines of the file:
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@@
 </segment>
 </net>
-<net name="SUIVEUR_IDC_SDA" class="0">
+<net name="SUIVEUR_I2C_SDA" class="0">
 <segment>
 <pinref part="MYRIO_PORT_A" gate="-34" pin="S"/>
